File: schematics/sat_ir_link/sat_ir_link.kicad_sch (KiCad schematic)
At the start: 19 parts, among them J1 Conn_01x05, J2 TSOP38238, Q1 2N2222

Commit message: New board circuits to fix design issues
Parts:
- removed J1: Conn_01x05, Connector_PinHeader_2.54mm:PinHeader_1x05_P2.54mm_Vertical, symbol Connector_Generic:Conn_01x05
- added J1: TX Connector, Connector:FanPinHeader_1x03_P2.54mm_Vertical, symbol Connector_Generic:Conn_01x03
- added J2: RX Connector, Connector:FanPinHeader_1x03_P2.54mm_Vertical, symbol Connector_Generic:Conn_01x03
- added TP7: TestPoint, TestPoint:TestPoint_THTPad_D4.0mm_Drill2.0mm, symbol Connector:TestPoint
- renumbered J2 to J3
Connections:
- net +3.3v: now also J2.1 (Pin_1)
- net +5V: now also J1.1 (Pin_1)
- net GND: now also J1.3 (Pin_3); no longer C3.2, C4.2, J3.2 (Pin_2)
- net RX_GPIO: now also J2.2 (Pin_2)
- net TX_GPIO: now also J1.2 (Pin_2)
- new net GND2: C3.2, C4.2, J2.3 (Pin_3), J3.2 (Pin_2), TP7.1
Other:
- moved on the sheet: TP1, TP3
